File: hw.kicad/scanner.sch (KiCad schematic (older format))
At the start: 25 parts

Commit message: fix compilation issues
Parts:
- removed K? (x25): RELAY_2RT, symbol RELAY_2RT
- added U? (x3): MIC5841, symbol MIC5841
Connections:
- net labels added: +5V, GND
- wire segments 0 -> 21
