File: hw.kicad/KeithleyUpgrade.kicad_pcb (KiCad board)
At the start: 2 copper layers, 85.1 x 65 mm, 78 parts, among them J1 DEBUG_PORT, J14 DISPLAY_BOARD, K1 TRIGGER, P1 TC2030-MCP, P18 CONN_8, P8 TP1, P9 TP1, Q1 BC850, U1 24AA256, U2 FT230x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

Commit message: fix compilation issues
Parts:
- removed REF** (x4): MountingHole_2-5mm, Mounting_Holes:MountingHole_2-5mm
- added R24: 220, Resistors_SMD:R_0805, F.Cu at (114.8, 89.2)
- P1: footprint Tag-Connect:TC2030_SMALL -> Tag-Connect:TC2030-NL_SMALL
- moved R14 9.19 mm to (120.4, 68.0), turned to 270 degrees
- moved C2 4.94 mm to (112.8, 100.8), turned to 180 degrees
- moved R1 3.16 mm to (118.1, 112.1)
- moved R2 3.15 mm to (114.2, 109.5), turned to 180 degrees
- moved J1 1.31 mm to (128.8, 121.5), turned to 0 degrees
- moved P1 1.31 mm to (135.6, 91.1)
- moved R3 0.94 mm to (114.2, 106.9), turned to 180 degrees
- moved P18 0.68 mm to (182.8, 76.6)
- moved C1 0.58 mm to (112.9, 103.2), turned to 180 degrees
- moved R4 0.45 mm to (107.8, 90.8)
Connections:
- net Net-(C1-Pad2) renamed /_usb+
- net Net-(C2-Pad2) renamed /_usb-
- net Net-(JP1-Pad2) renamed /usb+
- net Net-(JP1-Pad3) renamed /usb-
- net VCC renamed +5V
- U1 pad 7: GND -> /WP
- U3 pad 51: (no net) -> /WP
Routing:
- net /ADATA: track 5.08 -> 56.6 mm, vias 0 -> 2
- net /~CLOCK: track 46.7 -> 0.00 mm, vias 1 -> 0
- net /ACLOCK: track 5.61 -> 51.3 mm, vias 0 -> 2
- net Net-(J1-Pad3): track 0.00 -> 45.7 mm, vias 0 -> 1
- net GND: track 0.00 -> 42.0 mm, vias 0 -> 31
- net Net-(J1-Pad5): track 1.24 -> 43.1 mm
- net /RxD: track 0.00 -> 41.7 mm, vias 0 -> 2
- net Net-(J1-Pad1): track 0.00 -> 39.7 mm, vias 0 -> 1
- net Net-(J1-Pad2): track 0.00 -> 35.7 mm, vias 0 -> 1
- net Net-(R24-Pad1): track 0.00 -> 35.6 mm
- net /~ASTROBE: track 5.61 -> 41.2 mm, vias 0 -> 2
- net Net-(J1-Pad4): track 0.00 -> 34.5 mm, vias 0 -> 1
- net /TxD: track 0.00 -> 34.1 mm
- net Net-(J1-Pad6): track 0.00 -> 30.7 mm, vias 0 -> 1
- net /d1: track 0.00 -> 29.7 mm, vias 0 -> 2
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- added copper zone on In1.Cu, net GND
Other:
- board size 85.1 x 65 mm -> 85 x 60 mm
- copper layers 2 -> 4

Commit message: added a couple of nets to the pcb
Routing:
- net /st: track 0.00 -> 58.4 mm, vias 0 -> 2
- net /~CLOCK: track 0.00 -> 58.2 mm
- net /err: track 0.00 -> 49.5 mm, vias 0 -> 2
- net /ok: track 0.00 -> 46.4 mm, vias 0 -> 2
- net Net-(D5-Pad1): track 0.00 -> 2.09 mm
- net Net-(D6-Pad1): track 0.00 -> 2.04 mm
Changed lines of the file:
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@@
-(kicad_pcb (version 4) (host pcbnew no-vcs-found-product)
+(kicad_pcb (version 4) (host pcbnew 4.1.0-alpha+201605180746+6813~44~ubuntu16.04.1-product)
   (general
     (links 262)
-    (no_connects 150)
-    (area 93.519499 61.426 189.519695 126.3756)
+    (no_connects 128)
+    (area 93.519499 61.77652 186.993 125.3575)
     (thickness 1.6)
     (drawings 6)
-    (tracks 847)
+    (tracks 916)
     (zones 0)
     (modules 75)
@@
     (pad_to_mask_clearance 0)
     (aux_axis_origin 0 0)
-    (visible_elements FFFEF77F)
+    (visible_elements FFFEFF7F)
     (pcbplotparams
       (layerselection 0x00030_80000001)
@@
       (hpglpenspeed 20)
       (hpglpendiameter 15)
-      (hpglpenoverlay 2)
       (psnegative false)
       (psa4output false)
@@
   (segment (start 135.87 96.6811) (end 135.88092 96.69202) (width 0.16) (layer F.Cu) (net 7) (status 30))
   (segment (start 133.07 95.5) (end 135.87 95.5) (width 0.16) (layer B.Cu) (net 7))
-  (via (at 135.87 95.5) (size 0.6) (drill 0.35) (layers F.Cu B.Cu) (net 7))
+  (via (at 135.9281 95.4913) (size 0.6) (drill 0.35) (layers F.Cu B.Cu) (net 7))
   (segment (start 128.03 93.39) (end 130.14 95.5) (width 0.16) (layer F.Cu) (net 7))
   (segment (start 130.14 95.5) (end 133.07 95.5) (width 0.16) (layer F.Cu) (net 7))
@@
   (via (at 176.58 106.04) (size 0.6) (drill 0.35) (layers F.Cu B.Cu) (net 51))
   (segment (start 176.56 106.06) (end 176.58 106.04) (width 0.16) (layer F.Cu) (net 51))
+  (segment (start 140.1252 95.4339) (end 140.27766 95.58636) (width 0.16) (layer F.Cu) (net 52))
+  (segment (start 140.27766 95.58636) (end 140.27766 96.69202) (width 0.16) (layer F.Cu) (net 52))
+  (segment (start 140.1252 94.487612) (end 140.1252 95.4339) (width 0.16) (layer F.Cu) (net 52))
+  (segment (start 142.24 87.3633) (end 140.1252 89.4781) (width 0.16) (layer B.Cu) (net 52))
+  (via (at 140.1252 94.487612) (size 0.6) (drill 0.35) (layers F.Cu B.Cu) (net 52))
+  (segment (start 140.1252 89.4781) (end 140.1252 94.487612) (width 0.16) (layer B.Cu) (net 52))
+  (segment (start 163.50999 87.497448) (end 163.067437 87.940001) (width 0.16) (layer F.Cu) (net 52))
+  (segment (start 163.067437 87.940001) (end 149.740799 87.940001) (width 0.16) (layer F.Cu) (net 52))
+  (segment (start 149.740799 87.940001) (end 149.164098 87.3633) (width 0.16) (layer F.Cu) (net 52))
+  (segment (start 149.164098 87.3633) (end 142.24 87.3633) (width 0.16) (layer F.Cu) (net 52))
+  (via (at 142.24 87.3633) (size 0.6) (drill 0.35) (layers F.Cu B.Cu) (net 52))
+  (segment (start 163.50999 79.877448) (end 163.50999 87.497448) (width 0.16) (layer F.Cu) (net 52))
+  (segment (start 168.362438 75.025) (end 163.50999 79.877448) (width 0.16) (layer F.Cu) (net 52))
+  (segment (start 171.42598 75.025) (end 168.362438 75.025) (width 0.16) (layer F.Cu) (net 52))
   (segment (start 183.01 109.222) (end 182.762 109.222) (width 0.16) (layer B.Cu) (net 53) (status 30))
   (segment (start 182.762 109.222) (end 181.48 107.94) (width 0.16) (layer B.Cu) (net 53) (status 10))
@@
   (segment (start 178.707 116.842) (end 180.47 116.842) (width 0.16) (layer F.Cu) (net 60) (status 20))
   (segment (start 176.885 115.02) (end 178.707 116.842) (width 0.16) (layer F.Cu) (net 60))
+  (segment (start 140.6652 95.1484) (end 140.6652 96.67824) (width 0.16) (layer F.Cu) (net 61))
+  (segment (start 140.6652 96.67824) (end 140.67898 96.69202) (width 0.16) (layer F.Cu) (net 61))
+  (segment (start 140.97 90.17) (end 140.6652 90.4748) (width 0.16) (layer B.Cu) (net 61))
+  (segment (start 140.6652 90.4748) (end 140.6652 95.1484) (width 0.16) (layer B.Cu) (net 61))
+  (via (at 140.6652 95.1484) (size 0.6) (drill 0.35) (layers F.Cu B.Cu) (net 61))
+  (segment (start 142.24 88.9) (end 140.97 90.17) (width 0.16) (layer B.Cu) (net 61))
+  (segment (start 163.83 87.63) (end 162.56 88.9) (width 0.16) (layer F.Cu) (net 61))
+  (segment (start 162.56 88.9) (end 142.24 88.9) (width 0.16) (layer F.Cu) (net 61))
+  (via (at 142.24 88.9) (size 0.6) (drill 0.35) (layers F.Cu B.Cu) (net 61))
+  (segment (start 163.83 80.01) (end 163.83 87.63) (width 0.16) (layer F.Cu) (net 61))
+  (segment (start 165.375 78.465) (end 163.83 80.01) (width 0.16) (layer F.Cu) (net 61))
+  (segment (start 171.38598 78.465) (end 165.375 78.465) (width 0.16) (layer F.Cu) (net 61))
   (segment (start 174.855 111.21) (end 177.21 111.21) (width 0.16) (layer F.Cu) (net 62) (status 10))
   (segment (start 179.198 109.222) (end 180.47 109.222) (width 0.16) (layer F.Cu) (net 62) (status 20))
@@
   (segment (start 174.505 87.955) (end 176.865 87.955) (width 0.16) (layer F.Cu) (net 63) (status 20))
   (segment (start 173.235 86.685) (end 174.505 87.955) (width 0.16) (layer F.Cu) (net 63))
+  (segment (start 181.6735 104.8512) (end 181.6735 102.9385) (width 0.16) (layer F.Cu) (net 64))
+  (segment (start 181.6735 102.9385) (end 183.01 101.602) (width 0.16) (layer F.Cu) (net 64))
+  (segment (start 181.1147 105.41) (end 181.6735 104.8512) (width 0.16) (layer F.Cu) (net 64))
+  (segment (start 179.6161 105.41) (end 181.1147 105.41) (width 0.16) (layer F.Cu) (net 64))
+  (segment (start 178.8033 106.2228) (end 179.6161 105.41) (width 0.16) (layer F.Cu) (net 64))
+  (segment (start 178.8033 106.7181) (end 178.8033 106.2228) (width 0.16) (layer F.Cu) (net 64))
+  (segment (start 176.2252 109.2962) (end 178.8033 106.7181) (width 0.16) (layer F.Cu) (net 64))
+  (segment (start 165.5191 109.2962) (end 176.2252 109.2962) (width 0.16) (layer F.Cu) (net 64))
+  (segment (start 164.4142 110.4011) (end 165.5191 109.2962) (width 0.16) (layer F.Cu) (net 64))
+  (segment (start 146.1897 110.4011) (end 164.4142 110.4011) (width 0.16) (layer F.Cu) (net 64))
+  (segment (start 139.87888 104.09028) (end 146.1897 110.4011) (width 0.16) (layer F.Cu) (net 64))
+  (segment (start 139.87888 96.69202) (end 139.87888 104.09028) (width 0.16) (layer F.Cu) (net 64))
   (segment (start 139.877973 96.691113) (end 139.87888 96.69202) (width 0.16) (layer F.Cu) (net 64) (status 30))
   (segment (start 109.6 98.77) (end 109.6 98.332379) (width 0.16) (layer F.Cu) (net 65))
@@
   (segment (start 131.98202 100.19214) (end 127.23814 100.19214) (width 0.16) (layer F.Cu) (net 69))
   (segment (start 127.23814 100.19214) (end 127.22 100.174) (width 0.16) (layer F.Cu) (net 69))
+  (segment (start 173.48402 78.465) (end 175.575 78.465) (width 0.16) (layer F.Cu) (net 70))
+  (segment (start 173.52402 75.025) (end 175.5586 75.025) (width 0.16) (layer F.Cu) (net 71))
+  (segment (start 175.5586 75.025) (end 175.5656 75.032) (width 0.16) (layer F.Cu) (net 71))
   (segment (start 173.57402 71.455) (end 175.5358 71.455) (width 0.16) (layer F.Cu) (net 72) (status 30))
   (segment (start 175.5358 71.455) (end 175.5656 71.4252) (width 0.16) (layer F.Cu) (net 72) (status 30))
@@
   (segment (start 129.806234 98.001331) (end 125.758329 98.001331) (width 0.16) (layer F.Cu) (net 93))
   (segment (start 107.255 93.427562) (end 107.255 93.91) (width 0.16) (layer F.Cu) (net 93))
+  (segment (start 135.48214 96.69202) (end 135.48214 95.844542) (width 0.16) (layer F.Cu) (net 94))
+  (segment (start 135.388099 95.2333) (end 135.6614 94.959999) (width 0.16) (layer F.Cu) (net 94))
+  (segment (start 135.48214 95.844542) (end 135.388099 95.750501) (width 0.16) (layer F.Cu) (net 94))
+  (segment (start 135.388099 95.750501) (end 135.388099 95.2333) (width 0.16) (layer F.Cu) (net 94))
+  (segment (start 136.423599 94.959999) (end 135.6614 94.959999) (width 0.16) (layer F.Cu) (net 94))
+  (segment (start 135.6614 94.959999) (end 135.610799 94.959999) (width 0.16) (layer F.Cu) (net 94))
+  (segment (start 136.7536 95.29) (end 136.423599 94.959999) (width 0.16) (layer F.Cu) (net 94))
+  (segment (start 139.3444 95.3262) (end 139.080599 95.590001) (width 0.16) (layer B.Cu) (net 94))
+  (segment (start 139.080599 95.590001) (end 137.053601 95.590001) (width 0.16) (layer B.Cu) (net 94))
+  (segment (start 137.053601 95.590001) (end 136.7536 95.29) (width 0.16) (layer B.Cu) (net 94))
+  (via (at 136.7536 95.29) (size 0.6) (drill 0.35) (layers F.Cu B.Cu) (net 94))
+  (segment (start 139.3444 88.767836) (end 139.3444 95.3262) (width 0.16) (layer B.Cu) (net 94))
+  (segment (start 142.1638 86.3727) (end 141.739536 86.3727) (width 0.16) (layer B.Cu) (net 94))
+  (segment (start 141.739536 86.3727) (end 139.3444 88.767836) (width 0.16) (layer B.Cu) (net 94))
+  (segment (start 150.9903 85.5599) (end 142.9766 85.5599) (width 0.16) (layer F.Cu) (net 94))
+  (segment (start 142.9766 85.5599) (end 142.1638 86.3727) (width 0.16) (layer F.Cu) (net 94))
+  (via (at 142.1638 86.3727) (size 0.6) (drill 0.35) (layers F.Cu B.Cu) (net 94))
+  (segment (start 153.3779 85.5599) (end 150.9903 85.5599) (width 0.16) (layer F.Cu) (net 94))
+  (segment (start 163.1442 84.5185) (end 163.1442 79.790676) (width 0.16) (layer F.Cu) (net 94))
+  (segment (start 163.1442 87.3125) (end 163.1442 84.5185) (width 0.16) (layer F.Cu) (net 94))
+  (segment (start 163.1442 84.5185) (end 162.1028 85.5599) (width 0.16) (layer F.Cu) (net 94))
+  (segment (start 162.1028 85.5599) (end 153.3779 85.5599) (width 0.16) (layer F.Cu) (net 94))
+  (segment (start 163.1442 79.790676) (end 168.229885 74.704991) (width 0.16) (layer F.Cu) (net 94))
+  (segment (start 168.229885 74.704991) (end 169.16041 74.70499) (width 0.16) (layer F.Cu) (net 94))
+  (segment (start 169.16041 74.70499) (end 170.18 73.6854) (width 0.16) (layer F.Cu) (net 94))
+  (segment (start 170.18 73.6854) (end 170.18 71.99154) (width 0.16) (layer F.Cu) (net 94))
+  (segment (start 170.18 71.99154) (end 170.71654 71.455) (width 0.16) (layer F.Cu) (net 94))
+  (segment (start 170.71654 71.455) (end 171.47598 71.455) (width 0.16) (layer F.Cu) (net 94))
   (segment (start 135.48 108.71) (end 135.48 110.06) (width 0.16) (layer F.Cu) (net 95) (status 20))
   (segment (start 135.48 110.06) (end 135.49 110.07) (width 0.16) (layer F.Cu) (net 95) (status 30))

Commit message: addedd documentation@
Parts:
- moved R19 21.0 mm to (114.2, 114.2), turned to 179 degrees
- moved C21 11.9 mm to (155.6, 77.0), turned to 90 degrees
- moved R23 9.96 mm to (136.9, 86.8)
- moved C20 5.39 mm to (143.6, 78.1), turned to 90 degrees
- moved R1 3.86 mm to (114.2, 111.9), turned to 180 degrees
Routing:
- net Net-(R1-Pad1): track 3.75 -> 33.8 mm, vias 2 -> 3
- net /st: track 58.4 -> 37.6 mm
- net Net-(C3-Pad2): track 11.9 -> 30.9 mm
- net /err: track 49.5 -> 32.3 mm
- net /ok: track 46.4 -> 30.2 mm
- net +5V: track 0.00 -> 12.9 mm
- net Net-(JP1-Pad1): track 0.00 -> 4.43 mm
- net MCLR: track 8.43 -> 11.0 mm
- net GND: track 42.0 -> 40.4 mm, vias 31 -> 29
- added copper zone on F.Cu, net +3.3V
- added copper zone on B.Cu, net GND
- removed copper zone on In1.Cu, net GND
