File: hw.kicad/KeithleyUpgrade.sch (KiCad schematic (older format))
At the start: 72 parts, among them J1 DEBUG_PORT, J14 DISPLAY_BOARD, K1 TRIGGER, P1 PROG, P18 CONN_8, P8 TP1, P9 TP1, Q1 BC850, U1 24AA256, U2 FT230x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

Commit message: Adding files wrongly left out on last commit
Parts:
- added R?: 10k, symbol R
Connections:
- wire segments 404 -> 406
Other:
- moved on the sheet: P1

Commit message: implementing i2c
Connections:
- wire segments 406 -> 510
Other:
- moved on the sheet: U2

Commit message: fixed cristal footprint
Parts:
- added C22: 220u/10v, Capacitors_SMD:c_elec_10x10, symbol C
- C1, C10, C12, C14, C15, C16, C18, C19, C2, C20, C21, C3, C4, C6, C7, C8, C9: footprint (none) -> Capacitors_SMD:C_0805
- C11: footprint (none) -> Capacitors_SMD:c_elec_10x10
- C13, C17: footprint (none) -> Capacitors_SMD:C_1210
- C5: footprint (none) -> Capacitors_SMD:C_1206
- D1, D2, D3, D4: footprint (none) -> Diodes_SMD:Diode-SMA_Standard
- D5, D6, D7: footprint (none) -> LEDs:LED-0805
- J1, J14: footprint (none) -> personal:header_straight_2x13
- JP1: footprint (none) -> Connect:USB_B
- K1: footprint (none) -> Connect:bornier3
- L1: footprint (none) -> SMD_Packages:SMD-1210
- P1: footprint (none) -> Pin_Headers:Pin_Header_Straight_1x05
- P18: footprint (none) -> Pin_Headers:Pin_Header_Straight_1x08
- P8, P9: footprint (none) -> Connect:SIL-1
- Q1: footprint SOT-23 -> SMD_Packages:SOT23
- R1, R2, R3, R4, R5, R6, R7, R8: footprint (none) -> SMD_Packages:SM0805
- R10, R11, R12, R13, R14, R15, R16, R17, R18, R19, R20, R21, R22, R9: footprint (none) -> Resistors_SMD:R_0805
- R23: renamed from R?; footprint (none) -> Resistors_SMD:R_0805
- RP1, RP2: footprint (none) -> personal:SOM16
- SP1: footprint (none) -> Capacitors_Elko_ThroughHole:Elko_vert_DM14_RM5
- U1, U7: footprint (none) -> SOIC_Packages:SOIC-8_N
- U2: footprint qfn16 -> qfn:pvqfn-n16
- U3: footprint tqfp100 -> QFP:TQFP-100-4
- U4, U5: footprint (none) -> soic:soic-18
- U6: footprint (none) -> SMD_Packages:DPAK2
- U8: footprint (none) -> SOIC_Packages:SOIC-16_Narrow
- X1: footprint (none) -> personal:XTAL_SMD_5x3_2
Connections:
- wire segments 510 -> 408

Commit message: fixing format
Parts:
- C1, C10, C11, C12, C13, C14, C15, C16, C17, C18, C19, C2, C20, C21, C22, C3, C4, C5, C6, C7, C8, C9: symbol C -> C-RESCUE-KeithleyUpgrade
- D5, D6, D7: symbol LED -> LED-RESCUE-KeithleyUpgrade
- R1, R10, R11, R12, R13, R14, R15, R16, R17, R18, R19, R2, R20, R21, R22, R23, R3, R4, R5, R6, R7, R8, R9: symbol R -> R-RESCUE-KeithleyUpgrade
Connections:
- wire segments 408 -> 514

Commit message: updating schematic
Parts:
- removed P1: PROG, Pin_Headers:Pin_Header_Straight_1x05, symbol CONN_5
- added P1: TC2030-MCP, Tag-Connect:TC2030_SMALL, symbol TC2030-MCP
- U2: footprint qfn:pvqfn-n16 -> Housings_DFN_QFN:QFN-16-1EP_4x4mm_Pitch0.65mm
Connections:
- net +3.3V: now also P1.2 (Vdd)
- net GND: now also P1.3 (GND)
- net MCLR: now reaches R23.1, U3.13 (~MCLR)
- net MCLR: now also P1.1 (MCLR/Vpp)
- net PGC: now reaches U3.24 (PGEC1/RB1)
- net PGC: now also P1.5 (PGC)
- net PGD: now reaches U3.25 (PGED1/RB0)
- net PGD: now also P1.4 (PGD)
- net at U3.43 (RB14): now also J1.24 (P20)
- net at U3.44 (RB15): now also J1.26 (P22)

Commit message: fix compilation issues
Parts:
- added R24: 220, Resistors_SMD:R_0805, symbol R-RESCUE-KeithleyUpgrade
- P1: footprint Tag-Connect:TC2030_SMALL -> Tag-Connect:TC2030-NL_SMALL
Connections:
- net GND: no longer U1.7 (WP)
- net at U3.43 (RB14): now also J1.24 (P20)
- net at U3.44 (RB15): now also J1.26 (P22)
- net WP: now reaches U3.51 (RPF3/OC1)
- net WP: now also U1.7 (WP)
- net _usb-: now reaches C2.2, R3.1, U2.6 (USBDP)
- net _usb+: now reaches C1.2, R2.1, U2.7 (USBDM)
- net usb+: now reaches JP1.2 (D-), R2.2
- net usb-: now reaches JP1.3 (D+), R3.2
- net at Q1.3 (C), SP1.1: now also R24.2
- net at R7.2, SP1.2: now also R24.1
Other:
- moved on the sheet: R7

Commit message: addedd documentation@
Connections:
- net +3.3V: no longer R20.2, R21.2, R22.2
- net +5V: now also R20.2, R21.2, R22.2
- net at U3.43 (RB14): now also J1.24 (P20)
- net at U3.44 (RB15): now also J1.26 (P22)

Commit message: update documentation
Connections:
- net at U3.43 (RB14): now also J1.24 (P20)
- net at U3.44 (RB15): now also J1.26 (P22)
