File: hw.kicad/frontpanel/frontpanel.sch (KiCad schematic (older format))
At the start: 47 parts, among them U1 LTP-7357AG, U10 LTP-7357AG, U11 TLC5928, U12 TLC5928, U13 TLC5928, U14 TLC5928, U2 LTP-7357AG, U3 LTP-7357AG, U4 LTP-7357AG, U5 LTP-7357AG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

Commit message: update files
Parts:
- removed Q? (x7): Q_PMOS_DGS, symbol Q_PMOS_DGS
- removed Q? (x7): Q_NMOS_DGS, symbol Q_NMOS_DGS
- removed R? (x14): R, symbol R
- added P1, P2, P3, P4, P5, P6: CONN_10, Pin_Headers:Pin_Header_Straight_1x10, symbol CONN_10
- added P7, P8: CONN_8, Pin_Headers:Pin_Header_Straight_1x08, symbol CONN_8
- added U15: MIC2981, Housings_SOIC:SOIC-18_7.5x11.6mm_Pitch1.27mm, symbol MIC2981
- R1, R2, R3, R4: footprint (none) -> Resistors_SMD:R_0805
- U16: renamed from U?; footprint (none) -> Housings_DFN_QFN:QFN-28-1EP_6x6mm_Pitch0.65mm
Connections:
- net COL1: no longer U14.5 (CH0)
- net COL10: no longer U14.14 (CH9)
- net COL11: no longer U14.15 (CH10)
- net COL12: no longer U14.16 (CH11)
- net COL13: no longer U14.17 (CH12)
- net COL14: no longer U14.18 (CH13)
- net COL15: no longer U14.19 (CH14)
- net COL16: no longer U14.20 (CH15)
- net COL17: no longer U13.5 (CH0)
- net COL18: no longer U13.6 (CH1)
- net COL19: no longer U13.7 (CH2)
- net COL2: no longer U14.6 (CH1)
- net COL20: no longer U13.8 (CH3)
- net COL21: no longer U13.9 (CH4)
- net COL22: no longer U13.10 (CH5)
- net COL23: no longer U13.11 (CH6)
- net COL24: no longer U13.12 (CH7)
- net COL25: no longer U13.13 (CH8)
- net COL26: no longer U13.14 (CH9)
- net COL27: no longer U13.15 (CH10)
- net COL28: no longer U13.16 (CH11)
- net COL29: no longer U13.17 (CH12)
- net COL3: no longer U14.7 (CH2)
- net COL30: no longer U13.18 (CH13)
- net COL31: no longer U13.19 (CH14)
- net COL32: no longer U13.20 (CH15)
- net COL33: no longer U12.5 (CH0)
- net COL34: no longer U12.6 (CH1)
- net COL35: no longer U12.7 (CH2)
- net COL36: no longer U12.8 (CH3)
- net COL37: no longer U12.9 (CH4)
- net COL38: no longer U12.10 (CH5)
- net COL39: no longer U12.11 (CH6)
- net COL4: no longer U14.8 (CH3)
- net COL40: no longer U12.12 (CH7)
- net COL41: no longer U12.13 (CH8)
- net COL42: no longer U12.14 (CH9)
- net COL43: no longer U12.15 (CH10)
- net COL44: no longer U12.16 (CH11)
- net COL45: no longer U12.17 (CH12)
- net COL46: no longer U12.18 (CH13)
- net COL47: no longer U12.19 (CH14)
- net COL48: no longer U12.20 (CH15)
- net COL49: no longer U11.5 (CH0)
- net COL5: no longer U14.9 (CH4)
- net COL50: no longer U11.6 (CH1)
- net COL6: no longer U14.10 (CH5)
- net COL7: no longer U14.11 (CH6)
- net COL8: no longer U14.12 (CH7)
- net COL9: no longer U14.13 (CH8)
- net GND: now also U15.10 (VS)
- net VCC: now also U15.9 (VS)
Other:
- moved on the sheet: R1, R2, R3, R4, U11, U12, U13, U14, U16
